Commit message: Add collision geometry

File: src/oarbot_description/urdf/hokuyo/hokuyo_ust.urdf.xacro (robot description, xacro)
@@ -13,4 +13,11 @@
         <material name="clearpath_dark_grey" />
       </visual>
+      <collision>
+        <!-- Approximate the Hokuyo body with a simple box. -->
+        <origin xyz="0 0 0.035" rpy="0 0 0"/>
+        <geometry>
+          <box size="0.05 0.05 0.07"/>
+        </geometry>
+      </collision>
     </link>
     <link name="${name}_laser">
