Commit message: Add collision geometry

File: src/oarbot_description/urdf/custom/u_bracket.urdf.xacro (robot description, xacro)
@@ -129,4 +129,10 @@
         <material name="u_bracket_black"/>
       </visual>
+      <collision>
+        <origin xyz="0 0 0" rpy="0 1.5707963 0"/>
+        <geometry>
+          <cylinder radius="${mount_hole_radius}" length="${mount_hole_length}"/>
+        </geometry>
+      </collision>
     </link>
     <!-- ===== Mount reference frame: right wall ===== -->
@@ -144,4 +150,10 @@
         <material name="u_bracket_black"/>
       </visual>
+      <collision>
+        <origin xyz="0 0 0" rpy="0 1.5707963 0"/>
+        <geometry>
+          <cylinder radius="${mount_hole_radius}" length="${mount_hole_length}"/>
+        </geometry>
+      </collision>
     </link>
   </xacro:macro>
