Commit message: Add collision geometry

File: src/oarbot_description/urdf/custom/kinect_wrist_connection.urdf.xacro (robot description, xacro)
@@ -10,4 +10,12 @@
                 <material name="white" />
             </visual>
+            <collision>
+                <origin xyz="-0.05516 -0.0035 -0.025" rpy="0 0 0"/>
+                <geometry>
+                    <mesh
+                        scale="0.001 0.001 0.001"
+                        filename="package://oarbot_description/meshes/custom/wrist_connection.STL"/>
+                </geometry>
+            </collision>
             <inertial>
                 <origin xyz="0 0 0" rpy="0 0 0"/>
