Commit message: Add collision geometry

File: src/oarbot_description/urdf/microsoft/azure_kinect.urdf.xacro (robot description, xacro)
@@ -26,4 +26,10 @@
                 <material name="kinect_white" />
             </visual>
+            <collision>
+                <origin xyz="0. 0. 0." />
+                <geometry>
+                    <box size="0.0994 0.0996 0.023" />
+                </geometry>
+            </collision>
         </link>
         <link name="camera_base">
@@ -35,4 +41,10 @@
                 <material name="kinect_grey" />
             </visual>
+            <collision>
+                <origin xyz="-0.013 0. 0." />
+                <geometry>
+                    <box size="0.026 0.103 0.039" />
+                </geometry>
+            </collision>
         </link>
         <link name="camera_visor">
@@ -44,4 +56,10 @@
                 <material name="kinect_black" />
             </visual>
+            <collision>
+                <origin xyz="-0.0128 0. 0." />
+                <geometry>
+                    <box size="0.026 0.101 0.037" />
+                </geometry>
+            </collision>
         </link>
         <joint name="camera_base_to_body" type="fixed">
