Commit message: Add collision geometry

File: src/oarbot_description/urdf/microstrain/microstrain_imu.urdf.xacro (robot description, xacro)
@@ -10,4 +10,9 @@
         <material name="clearpath_dark_grey" />
       </visual>
+      <collision>
+        <geometry>
+          <box size="0.02 0.02 0.005"/>
+        </geometry>
+      </collision>
     </link>
     <joint name="${name}_base_joint" type="fixed">
