Commit message: Add frame prefix to robot description
This will allow us to use this description for the real robot

File: src/oarbot_description/urdf/clearpath/do100/do100.urdf.xacro (robot description, xacro)
@@ -6,5 +6,5 @@
   <xacro:property name="PI" value="${math.pi}" />
   <!-- D0100 Platform Macro -->
-  <xacro:macro name="do100" params="control:='omni_4wd' front_wheels:='mecanum' rear_wheels:='mecanum'">
+  <xacro:macro name="do100" params="prefix control:='omni_4wd' front_wheels:='mecanum' rear_wheels:='mecanum'">
     <!-- Variables -->
     <xacro:property name="wheelbase" value="0.570" />
@@ -13,11 +13,11 @@
     <xacro:property name="dummy_inertia" value="1e-09"/>
     <!-- Chassis -->
-    <link name="base_link"></link>
-    <joint name="base_link_joint" type="fixed">
+    <link name="${prefix}base_link"></link>
+    <joint name="${prefix}base_link_joint" type="fixed">
       <origin xyz="0 0 0" rpy="0 0 0" />
-      <parent link="base_link"/>
-      <child link="chassis_link" />
+      <parent link="${prefix}base_link"/>
+      <child link="${prefix}chassis_link" />
     </joint>
-    <link name="chassis_link">
+    <link name="${prefix}chassis_link">
       <visual>
         <origin xyz="0 0 0" rpy="0 0 0"/>
@@ -45,5 +45,5 @@
     <!-- Add wheels -->
     <xacro:include filename="$(find oarbot_description)/urdf/clearpath/do100/drivetrain/wheels.urdf.xacro"/>
-    <xacro:do100_drivetrain_wheels front_wheels="${front_wheels}" rear_wheels="${rear_wheels}"/>
+    <xacro:do100_drivetrain_wheels prefix="${prefix}" front_wheels="${front_wheels}" rear_wheels="${rear_wheels}"/>
     <!-- Add drivetrain -->
     <xacro:include filename="$(find oarbot_description)/urdf/clearpath/generic/drivetrain/drivetrain.urdf.xacro"/>
@@ -59,4 +59,5 @@
     </xacro:unless>
     <xacro:generic_drivetrain
+      prefix="${prefix}"
       name="do100"
       control="${control}"
@@ -66,5 +67,5 @@
     />
     <!-- Internal IMU -->
-    <link name="imu_0_link">
+    <link name="${prefix}imu_0_link">
       <inertial>
         <mass value="0.001"/>
@@ -73,10 +74,10 @@
       </inertial>
     </link>
-    <joint name="imu_joint" type="fixed">
-      <parent link="chassis_link" />
-      <child link="imu_0_link" />
+    <joint name="${prefix}imu_joint" type="fixed">
+      <parent link="${prefix}chassis_link" />
+      <child link="${prefix}imu_0_link" />
     </joint>
-    <gazebo reference="imu_0_link">
-      <sensor type="imu" name="imu_0">
+    <gazebo reference="${prefix}imu_0_link">
+      <sensor type="imu" name="${prefix}imu_0">
         <always_on>true</always_on>
         <update_rate>50</update_rate>
@@ -87,58 +88,58 @@
     </gazebo>
     <!-- Mounting Hard Points -->
-    <link name="default_mount"/>
-    <link name="front_2_mount"/>
-    <link name="front_1_mount"/>
-    <link name="front_0_mount"/>
-    <link name="rear_2_mount"/>
-    <link name="rear_1_mount"/>
-    <link name="rear_0_mount"/>
-    <joint name="default_mount_joint" type="fixed">
+    <link name="${prefix}default_mount"/>
+    <link name="${prefix}front_2_mount"/>
+    <link name="${prefix}front_1_mount"/>
+    <link name="${prefix}front_0_mount"/>
+    <link name="${prefix}rear_2_mount"/>
+    <link name="${prefix}rear_1_mount"/>
+    <link name="${prefix}rear_0_mount"/>
+    <joint name="${prefix}default_mount_joint" type="fixed">
       <origin xyz="0 0 0.069023" rpy="0 0 0" />
-      <parent link="chassis_link"/>
-      <child link="default_mount" />
+      <parent link="${prefix}chassis_link"/>
+      <child link="${prefix}default_mount" />
     </joint>
-    <joint name="front_0_mount_joint" type="fixed">
+    <joint name="${prefix}front_0_mount_joint" type="fixed">
       <origin xyz="0.080 0 0" rpy="0 0 0" />
-      <parent link="default_mount"/>
-      <child link="front_0_mount" />
+      <parent link="${prefix}default_mount"/>
+      <child link="${prefix}front_0_mount" />
     </joint>
-    <joint name="front_1_mount_joint" type="fixed">
+    <joint name="${prefix}front_1_mount_joint" type="fixed">
       <origin xyz="0.080 0 0" rpy="0 0 0" />
-      <parent link="front_0_mount"/>
-      <child link="front_1_mount" />
+      <parent link="${prefix}front_0_mount"/>
+      <child link="${prefix}front_1_mount" />
     </joint>
-    <joint name="front_2_mount_joint" type="fixed">
+    <joint name="${prefix}front_2_mount_joint" type="fixed">
       <origin xyz="0.080 0 0" rpy="0 0 0" />
-      <parent link="front_1_mount"/>
-      <child link="front_2_mount" />
+      <parent link="${prefix}front_1_mount"/>
+      <child link="${prefix}front_2_mount" />
     </joint>
-    <joint name="rear_0_mount_joint" type="fixed">
+    <joint name="${prefix}rear_0_mount_joint" type="fixed">
       <origin xyz="-0.080 0 0" rpy="0 0 0" />
-      <parent link="default_mount"/>
-      <child link="rear_0_mount" />
+      <parent link="${prefix}default_mount"/>
+      <child link="${prefix}rear_0_mount" />
     </joint>
-    <joint name="rear_1_mount_joint" type="fixed">
+    <joint name="${prefix}rear_1_mount_joint" type="fixed">
       <origin xyz="-0.080 0 0" rpy="0 0 0" />
-      <parent link="rear_0_mount"/>
-      <child link="rear_1_mount" />
+      <parent link="${prefix}rear_0_mount"/>
+      <child link="${prefix}rear_1_mount" />
     </joint>
-    <joint name="rear_2_mount_joint" type="fixed">
+    <joint name="${prefix}rear_2_mount_joint" type="fixed">
       <origin xyz="-0.080 0 0" rpy="0 0 0" />
-      <parent link="rear_1_mount"/>
-      <child link="rear_2_mount" />
+      <parent link="${prefix}rear_1_mount"/>
+      <child link="${prefix}rear_2_mount" />
     </joint>
     <!-- Bumper Mounts -->
-    <link name="front_bumper_mount"/>
-    <link name="rear_bumper_mount"/>
-    <joint name="front_bumper_mount_joint" type="fixed">
+    <link name="${prefix}front_bumper_mount"/>
+    <link name="${prefix}rear_bumper_mount"/>
+    <joint name="${prefix}front_bumper_mount_joint" type="fixed">
       <origin xyz="0.34159 0 0.0345115" rpy="0 0 0" />
-      <parent link="chassis_link"/>
-      <child link="front_bumper_mount" />
+      <parent link="${prefix}chassis_link"/>
+      <child link="${prefix}front_bumper_mount" />
     </joint>
-    <joint name="rear_bumper_mount_joint" type="fixed">
+    <joint name="${prefix}rear_bumper_mount_joint" type="fixed">
       <origin xyz="-0.34159 0 0.0345115" rpy="0 0 0" />
-      <parent link="chassis_link"/>
-      <child link="rear_bumper_mount" />
+      <parent link="${prefix}chassis_link"/>
+      <child link="${prefix}rear_bumper_mount" />
     </joint>
   </xacro:macro>

File: src/oarbot_description/urdf/clearpath/do100/drivetrain/wheels.urdf.xacro (robot description, xacro)
@@ -1,5 +1,5 @@
 <?xml version="1.0"?>
 <robot xmlns:xacro="http://ros.org/wiki/xacro" xmlns:gz="http://gazebosim.org/schema" name="do100_drivetrain_wheels">
-  <xacro:macro name="do100_drivetrain_wheels" params="front_wheels rear_wheels">
+  <xacro:macro name="do100_drivetrain_wheels" params="prefix front_wheels rear_wheels">
     <xacro:include filename="$(find oarbot_description)/urdf/clearpath/do100/drivetrain/wheels/mecanum.urdf.xacro"/>
     <!-- Front Wheels -->
@@ -7,8 +7,8 @@
       <xacro:property name="front_wheel_radius" value="${do100_mecanum_wheel_radius}" scope="parent"/>
       <xacro:property name="front_wheel_width" value="${do100_mecanum_wheel_width}" scope="parent"/>
-      <xacro:do100_mecanum_wheel prefix="front_left" side="-1">
+      <xacro:do100_mecanum_wheel prefix="front_left" tf_prefix="${prefix}" side="-1">
         <origin xyz="${wheelbase/2} ${track/2+front_wheel_width/2} ${wheel_vertical_offset}" rpy="0 0 0" />
       </xacro:do100_mecanum_wheel>
-      <xacro:do100_mecanum_wheel prefix="front_right" side="1">
+      <xacro:do100_mecanum_wheel prefix="front_right" tf_prefix="${prefix}" side="1">
         <origin xyz="${wheelbase/2} ${-track/2-front_wheel_width/2} ${wheel_vertical_offset}" rpy="0 0 0" />
       </xacro:do100_mecanum_wheel>
@@ -21,8 +21,8 @@
       <xacro:property name="rear_wheel_radius" value="${do100_mecanum_wheel_radius}" scope="parent"/>
       <xacro:property name="rear_wheel_width" value="${do100_mecanum_wheel_width}" scope="parent"/>
-      <xacro:do100_mecanum_wheel prefix="rear_left" side="1">
+      <xacro:do100_mecanum_wheel prefix="rear_left" tf_prefix="${prefix}" side="1">
         <origin xyz="${-wheelbase/2} ${track/2+rear_wheel_width/2} ${wheel_vertical_offset}" rpy="0 0 0" />
       </xacro:do100_mecanum_wheel>
-      <xacro:do100_mecanum_wheel prefix="rear_right" side="-1">
+      <xacro:do100_mecanum_wheel prefix="rear_right" tf_prefix="${prefix}" side="-1">
         <origin xyz="${-wheelbase/2} ${-track/2-rear_wheel_width/2} ${wheel_vertical_offset}" rpy="0 0 0" />
       </xacro:do100_mecanum_wheel>

File: src/oarbot_description/urdf/clearpath/do100/drivetrain/wheels/mecanum.urdf.xacro (robot description, xacro)
@@ -4,6 +4,6 @@
   <xacro:property name="do100_mecanum_wheel_mass" value="0.4" />
   <xacro:property name="do100_mecanum_wheel_width" value="0.050" />
-  <xacro:macro name="do100_mecanum_wheel" params="prefix side *joint_pose">
-    <link name="${prefix}_wheel_link">
+  <xacro:macro name="do100_mecanum_wheel" params="prefix tf_prefix side *joint_pose">
+    <link name="${tf_prefix}${prefix}_wheel_link">
       <visual>
         <origin xyz="0 ${side * 0.027} 0" rpy="0 0 ${PI/2}"/>
@@ -29,5 +29,5 @@
     <gazebo>
       <plugin filename="libgz-sim-wheel-slip-system.so" name="gz::sim::systems::WheelSlip">
-        <wheel link_name="${prefix}_wheel_link">
+        <wheel link_name="${tf_prefix}${prefix}_wheel_link">
           <slip_compliance_lateral>1.0</slip_compliance_lateral>
           <slip_compliance_longitudinal>1.0</slip_compliance_longitudinal>
@@ -37,5 +37,5 @@
       </plugin>
     </gazebo>
-    <gazebo reference="${prefix}_wheel_link">
+    <gazebo reference="${tf_prefix}${prefix}_wheel_link">
       <collision>
         <surface>
@@ -50,7 +50,7 @@
       </collision>
     </gazebo>
-    <joint name="${prefix}_wheel_joint" type="continuous">
-      <parent link="chassis_link"/>
-      <child link="${prefix}_wheel_link" />
+    <joint name="${tf_prefix}${prefix}_wheel_joint" type="continuous">
+      <parent link="${tf_prefix}chassis_link"/>
+      <child link="${tf_prefix}${prefix}_wheel_link" />
       <xacro:insert_block name="joint_pose" />
       <axis xyz="0 1 0" />

File: src/oarbot_description/urdf/clearpath/generic/drivetrain/control/omni_4wd.urdf.xacro (robot description, xacro)
@@ -1,5 +1,5 @@
 <?xml version="1.0"?>
 <robot xmlns:xacro="http://ros.org/wiki/xacro" xmlns:gz="http://gazebosim.org/schema" name="generic_drivetrain_control_omni_4wd">
-  <xacro:macro name="generic_drivetrain_control_omni_4wd" params="name hardware_plugin">
+  <xacro:macro name="generic_drivetrain_control_omni_4wd" params="prefix name hardware_plugin">
     <!-- Gazebo Controller -->
     <!-- <xacro:include filename="$(find oarbot_description)/urdf/clearpath/generic/gazebo.urdf.xacro"/> -->

File: src/oarbot_description/urdf/clearpath/generic/drivetrain/drivetrain.urdf.xacro (robot description, xacro)
@@ -1,9 +1,9 @@
 <?xml version="1.0"?>
 <robot xmlns:xacro="http://ros.org/wiki/xacro" xmlns:gz="http://gazebosim.org/schema" name="generic_drivetrain">
-  <xacro:macro name="generic_drivetrain" params="name control front_wheels rear_wheels hardware_plugin">
+  <xacro:macro name="generic_drivetrain" params="prefix name control front_wheels rear_wheels hardware_plugin">
     <!-- Omni drivetrain -->
     <xacro:if value="${control == 'omni_4wd'}">
       <xacro:include filename="$(find oarbot_description)/urdf/clearpath/generic/drivetrain/control/omni_4wd.urdf.xacro"/>
-      <xacro:generic_drivetrain_control_omni_4wd name="${name}" hardware_plugin="${hardware_plugin}"/>
+      <xacro:generic_drivetrain_control_omni_4wd prefix="${prefix}" name="${name}" hardware_plugin="${hardware_plugin}"/>
     </xacro:if>
     <!-- Diff 4WD drivetrain -->

File: src/oarbot_description/urdf/custom/kinect_wrist_connection.urdf.xacro (robot description, xacro)
@@ -1,6 +1,6 @@
 <?xml version="1.0"?>
 <robot xmlns:xacro="http://www.ros.org/wiki/xacro" name="kinect_wrist_connection">
-    <xacro:macro name="kinect_wrist_connection" params="num parent_link *origin">
-        <link name="wrist_connection_${num}_link">
+    <xacro:macro name="kinect_wrist_connection" params="num parent_link prefix *origin">
+        <link name="${prefix}wrist_connection_${num}_link">
             <visual>
                 <origin xyz="-0.05516 -0.0035 -0.025" rpy="0 0 0"/>
@@ -27,8 +27,8 @@
             </inertial>
         </link>
-        <joint name="wrist_connection_${num}_joint" type="fixed">
+        <joint name="${prefix}wrist_connection_${num}_joint" type="fixed">
             <xacro:insert_block name="origin"/>
             <parent link="${parent_link}"/>
-            <child link="wrist_connection_${num}_link"/>
+            <child link="${prefix}wrist_connection_${num}_link"/>
         </joint>
     </xacro:macro>

File: src/oarbot_description/urdf/custom/robot_arm_riser.urdf.xacro (robot description, xacro)
@@ -1,7 +1,7 @@
 <?xml version="1.0"?>
 <robot xmlns:xacro="http://www.ros.org/wiki/xacro" name="robot_arm_riser">
-    <xacro:macro name="robot_arm_riser" params="parent">
+    <xacro:macro name="robot_arm_riser" params="prefix parent">
         <!-- PVC RISER LINK -->
-        <link name="robot_arm_riser_link">
+        <link name="${prefix}robot_arm_riser_link">
             <visual>
                 <origin xyz="0 0 0.003175" rpy="0 0 0" />
@@ -30,19 +30,19 @@
             </inertial>
         </link>
-        <joint name="robot_arm_riser_joint" type="fixed">
+        <joint name="${prefix}robot_arm_riser_joint" type="fixed">
             <parent link="${parent}" />
-            <child link="robot_arm_riser_link" />
+            <child link="${prefix}robot_arm_riser_link" />
             <origin xyz="0 0 0" rpy="0 0 0" />
         </joint>
         <!-- ADD A LINK TO SPECIFY THE ARM MOUNT FRAME POSE -->
-        <link name="arm_mount" />
+        <link name="${prefix}arm_mount" />
         <!-- AND SPECIFY WHERE IS IT -->
-        <joint name="arm_mount_joint" type="fixed">
+        <joint name="${prefix}arm_mount_joint" type="fixed">
             <origin xyz="0 0 0.579525" rpy="0 0 0" />
-            <parent link="robot_arm_riser_link" />
-            <child link="arm_mount" />
+            <parent link="${prefix}robot_arm_riser_link" />
+            <child link="${prefix}arm_mount" />
         </joint>
         <!-- PVC RISER ARUCO MOUNT LINK -->
-        <link name="robot_arm_riser_aruco_mount_link">
+        <link name="${prefix}robot_arm_riser_aruco_mount_link">
             <visual>
                 <origin xyz="0 0 0" rpy="0 0 0" />
@@ -71,11 +71,11 @@
             </inertial>
         </link>
-        <joint name="robot_arm_riser_aruco_mount_joint" type="fixed">
+        <joint name="${prefix}robot_arm_riser_aruco_mount_joint" type="fixed">
             <parent link="${parent}" />
-            <child link="robot_arm_riser_aruco_mount_link" />
+            <child link="${prefix}robot_arm_riser_aruco_mount_link" />
             <origin xyz="0 0 0.503175" rpy="0 0 0" />
         </joint>
         <!-- PVC RISER UWB MOUNT LINK -->
-        <link name="robot_arm_riser_uwb_mount_link">
+        <link name="${prefix}robot_arm_riser_uwb_mount_link">
             <visual>
                 <origin xyz="0 0 0" rpy="0 0 0" />
@@ -104,7 +104,7 @@
             </inertial>
         </link>
-        <joint name="robot_arm_riser_uwb_mount_joint" type="fixed">
+        <joint name="${prefix}robot_arm_riser_uwb_mount_joint" type="fixed">
             <parent link="${parent}" />
-            <child link="robot_arm_riser_uwb_mount_link" />
+            <child link="${prefix}robot_arm_riser_uwb_mount_link" />
             <origin xyz="0 0 0.573175" rpy="0 0 0" />
         </joint>

File: src/oarbot_description/urdf/custom/u_bracket.urdf.xacro (robot description, xacro)
@@ -58,11 +58,11 @@
     <color rgba="0.05 0.05 0.05 1.0"/>
   </material>
-  <xacro:macro name="u_bracket" params="parent *origin">
-    <joint name="parent_to_u_bracket" type="fixed">
+  <xacro:macro name="u_bracket" params="parent prefix *origin">
+    <joint name="${prefix}parent_to_u_bracket" type="fixed">
       <xacro:insert_block name="origin"/>
       <parent link="${parent}"/>
-      <child link="u_bracket"/>
+      <child link="${prefix}u_bracket"/>
     </joint>
-    <link name="u_bracket">
+    <link name="${prefix}u_bracket">
       <!-- ===== Base of the U ===== -->
       <visual>
@@ -116,10 +116,10 @@
     </link>
     <!-- ===== Mount reference frame: left wall ===== -->
-    <joint name="left_mount_joint" type="fixed">
+    <joint name="${prefix}left_mount_joint" type="fixed">
       <origin xyz="${-wall_x_offset} 0 ${wall_z_center}" rpy="0 0 0"/>
-      <parent link="u_bracket"/>
-      <child link="left_mount"/>
+      <parent link="${prefix}u_bracket"/>
+      <child link="${prefix}left_mount"/>
     </joint>
-    <link name="left_mount">
+    <link name="${prefix}left_mount">
       <visual>
         <origin xyz="0 0 0" rpy="0 1.5707963 0"/>
@@ -137,10 +137,10 @@
     </link>
     <!-- ===== Mount reference frame: right wall ===== -->
-    <joint name="right_mount_joint" type="fixed">
+    <joint name="${prefix}right_mount_joint" type="fixed">
       <origin xyz="${wall_x_offset} 0 ${wall_z_center}" rpy="0 0 0"/>
-      <parent link="u_bracket"/>
-      <child link="right_mount"/>
+      <parent link="${prefix}u_bracket"/>
+      <child link="${prefix}right_mount"/>
     </joint>
-    <link name="right_mount">
+    <link name="${prefix}right_mount">
       <visual>
         <origin xyz="0 0 0" rpy="0 1.5707963 0"/>

File: src/oarbot_description/urdf/custom/uwb_tag.urdf.xacro (robot description, xacro)
@@ -1,6 +1,6 @@
 <?xml version="1.0"?>
 <robot xmlns:xacro="http://www.ros.org/wiki/xacro" name="uwb_tag">
-    <xacro:macro name="uwb_tag" params="tag_num parent *joint_pose">
-        <link name="uwb_tag_${tag_num}_link">
+    <xacro:macro name="uwb_tag" params="tag_num parent prefix *joint_pose">
+        <link name="${prefix}uwb_tag_${tag_num}_link">
             <visual>
                 <origin xyz="0 0 0" rpy="0 0 0"/>
@@ -25,7 +25,7 @@
             </inertial>
         </link>
-        <joint name="uwb_tag_${tag_num}_joint" type="fixed">
+        <joint name="${prefix}uwb_tag_${tag_num}_joint" type="fixed">
             <parent link="${parent}"/>
-            <child link="uwb_tag_${tag_num}_link" />
+            <child link="${prefix}uwb_tag_${tag_num}_link" />
             <xacro:insert_block name="joint_pose" />
         </joint>

File: src/oarbot_description/urdf/hokuyo/hokuyo_ust.urdf.xacro (robot description, xacro)
@@ -1,8 +1,8 @@
 <?xml version="1.0"?>
 <robot xmlns:xacro="http://ros.org/wiki/xacro">
-  <xacro:macro name="hokuyo_ust" params="name parent_link *origin
+  <xacro:macro name="hokuyo_ust" params="name parent_link prefix *origin
                                           ang_res:=0.25 min_ang:=-2.35619 max_ang:=2.35619
                                           update_rate:=40 min_range:=0.06 max_range:=30.0">
-    <link name="${name}_link">
+    <link name="${prefix}${name}_link">
       <visual>
         <origin xyz="0 0 0" rpy="0 0 0" />
@@ -21,5 +21,5 @@
       </collision>
     </link>
-    <link name="${name}_laser">
+    <link name="${prefix}${name}_laser">
       <inertial>
         <mass value="1.1" />
@@ -30,18 +30,18 @@
       </inertial>
     </link>
-    <joint name="${name}_joint" type="fixed">
+    <joint name="${prefix}${name}_joint" type="fixed">
       <xacro:insert_block name="origin" />
       <parent link="${parent_link}" />
-      <child link="${name}_link" />
+      <child link="${prefix}${name}_link" />
     </joint>
-    <joint name="${name}_laser_joint" type="fixed">
+    <joint name="${prefix}${name}_laser_joint" type="fixed">
       <!-- This offset is from the base of the bracket to the LIDAR's focal point. -->
       <origin xyz="0 0 0.0474" rpy="0 0 0" />
-      <parent link="${name}_link" />
-      <child link="${name}_laser" />
+      <parent link="${prefix}${name}_link" />
+      <child link="${prefix}${name}_laser" />
     </joint>
     <xacro:property name="samples" value="${round((max_ang - min_ang) * 180 / (ang_res * pi))}"/>
-    <gazebo reference="${name}_laser">
-      <sensor name="${name}" type="gpu_lidar">
+    <gazebo reference="${prefix}${name}_laser">
+      <sensor name="${prefix}${name}" type="gpu_lidar">
         <update_rate>${update_rate}</update_rate>
         <visualize>true</visualize>

File: src/oarbot_description/urdf/microsoft/azure_kinect.urdf.xacro (robot description, xacro)
@@ -5,5 +5,5 @@
  -->
 <robot name="azure-kinect" xmlns:xacro="http://www.ros.org/wiki/xacro">
-    <xacro:macro name="azure_kinect" params="parent_link *origin">
+    <xacro:macro name="azure_kinect" params="parent_link prefix *origin">
         <material name="kinect_black">
             <color rgba="0. 0. 0. 1" />
@@ -18,5 +18,5 @@
             <color rgba="0.9 0.9 0.9 1" />
         </material>
-        <link name="camera_body">
+        <link name="${prefix}camera_body">
             <visual>
                 <origin xyz="0. 0. 0." />
@@ -33,5 +33,5 @@
             </collision>
         </link>
-        <link name="camera_base">
+        <link name="${prefix}camera_base">
             <visual>
                 <origin xyz="-0.013 0. 0." />
@@ -48,5 +48,5 @@
             </collision>
         </link>
-        <link name="camera_visor">
+        <link name="${prefix}camera_visor">
             <visual>
                 <origin xyz="-0.0128 0. 0." />
@@ -63,18 +63,18 @@
             </collision>
         </link>
-        <joint name="camera_base_to_body" type="fixed">
-            <parent link="camera_base" />
-            <child link="camera_body" />
+        <joint name="${prefix}camera_base_to_body" type="fixed">
+            <parent link="${prefix}camera_base" />
+            <child link="${prefix}camera_body" />
             <origin xyz="-0.0757 0. 0.008" rpy="0. 0. 0." />
         </joint>
-        <joint name="camera_base_to_visor" type="fixed">
-            <parent link="camera_base" />
-            <child link="camera_visor" />
+        <joint name="${prefix}camera_base_to_visor" type="fixed">
+            <parent link="${prefix}camera_base" />
+            <child link="${prefix}camera_visor" />
             <origin xyz="0. 0. 0." rpy="0. 0. 0." />
         </joint>
-        <joint name="parent_to_camera_base" type="fixed">
+        <joint name="${prefix}parent_to_camera_base" type="fixed">
             <xacro:insert_block name="origin" />
             <parent link="${parent_link}" />
-            <child link="camera_base" />
+            <child link="${prefix}camera_base" />
         </joint>
     </xacro:macro>
