Commit message: Add frame prefix to robot description
This will allow us to use this description for the real robot

File: src/oarbot_description/urdf/microstrain/microstrain_imu.urdf.xacro (robot description, xacro)
@@ -1,7 +1,7 @@
 <?xml version="1.0"?>
 <robot xmlns:xacro="http://ros.org/wiki/xacro">
-  <xacro:macro name="microstrain_imu" params="name parent_link update_rate:=100 *origin">
-    <link name="${name}_base_link"/>
-    <link name="${name}_link">
+  <xacro:macro name="microstrain_imu" params="name prefix parent_link update_rate:=100 *origin">
+    <link name="${prefix}${name}_base_link"/>
+    <link name="${prefix}${name}_link">
       <visual>
         <geometry>
@@ -16,16 +16,16 @@
       </collision>
     </link>
-    <joint name="${name}_base_joint" type="fixed">
+    <joint name="${prefix}${name}_base_joint" type="fixed">
       <xacro:insert_block name="origin" />
       <parent link="${parent_link}" />
-      <child link="${name}_base_link" />
+      <child link="${prefix}${name}_base_link" />
     </joint>
     <joint name="${name}_joint" type="fixed">
       <origin xyz="0 0 0.0025"/>
-      <parent link="${name}_base_link" />
-      <child link="${name}_link" />
+      <parent link="${prefix}${name}_base_link" />
+      <child link="${prefix}${name}_link" />
     </joint>
     <gazebo reference="${name}_link">
-      <sensor type="imu" name="${name}">
+      <sensor type="imu" name="${prefix}${name}">
         <always_on>true</always_on>
         <update_rate>${update_rate}</update_rate>

File: src/oarbot_description/urdf/oarbot_silver.urdf.xacro (robot description, xacro)
@@ -10,27 +10,28 @@
     <material name="cyan"><color rgba="0 1.0 1.0 1.0"/></material>
     <material name="clearpath_dark_grey"><color rgba="0.2 0.2 0.2 1.0" /></material>
+    <xacro:property name="prefix" value="oarbot_silver/" />
     <!-- Dingo base -->
     <xacro:include filename="$(find oarbot_description)/urdf/clearpath/do100/do100.urdf.xacro"/>
-    <xacro:do100 control="omni_4wd" front_wheels="mecanum" rear_wheels="mecanum"/>
+    <xacro:do100 prefix="${prefix}" control="omni_4wd" front_wheels="mecanum" rear_wheels="mecanum"/>
     <!-- PVC Robot Arm Riser -->
     <xacro:include filename="$(find oarbot_description)/urdf/custom/robot_arm_riser.urdf.xacro"/>
-    <xacro:robot_arm_riser parent="front_1_mount"/>
+    <xacro:robot_arm_riser prefix="${prefix}" parent="${prefix}front_1_mount"/>
     <!-- Kinova arm -->
     <xacro:include filename="$(find oarbot_description)/urdf/kinova/j2n6s300_with_force_torque.urdf.xacro"/>
-    <link name="rotate_arm_mount"></link>
-    <joint name="rotate_arm_mount_joint" type="fixed">
+    <link name="${prefix}rotate_arm_mount"></link>
+    <joint name="${prefix}rotate_arm_mount_joint" type="fixed">
         <origin xyz="0 0 0" rpy="0 0 ${PI}"/>
-        <parent link="arm_mount" />
-        <child link="rotate_arm_mount" />
+        <parent link="${prefix}arm_mount" />
+        <child link="${prefix}rotate_arm_mount" />
     </joint>
-    <xacro:j2n6s300  base_parent="rotate_arm_mount"/>
+    <xacro:j2n6s300 prefix="${prefix}j2n6s300" base_parent="${prefix}rotate_arm_mount"/>
     <!--  UWB Tags -->
     <xacro:include filename="$(find oarbot_description)/urdf/custom/uwb_tag.urdf.xacro"/>
     <!-- Right UWB Tag -->
-    <xacro:uwb_tag tag_num="1" parent="robot_arm_riser_uwb_mount_link">
+    <xacro:uwb_tag prefix="${prefix}" tag_num="1" parent="${prefix}robot_arm_riser_uwb_mount_link">
         <origin xyz="0.02 -0.224 -0.025" rpy="${PI/2} ${-PI/2} 0"/>
     </xacro:uwb_tag>
     <!-- Left UWB Tag -->
-    <xacro:uwb_tag tag_num="2" parent="robot_arm_riser_uwb_mount_link">
+    <xacro:uwb_tag prefix="${prefix}" tag_num="2" parent="${prefix}robot_arm_riser_uwb_mount_link">
         <origin xyz="-0.02 0.224 -0.025" rpy="${-PI/2} ${-PI/2} 0"/>
     </xacro:uwb_tag>
@@ -38,16 +39,16 @@
     <xacro:include filename="$(find oarbot_description)/urdf/custom/u_bracket.urdf.xacro"/>
     <xacro:include filename="$(find oarbot_description)/urdf/custom/kinect_wrist_connection.urdf.xacro"/>
-    <xacro:u_bracket parent="j2n6s300_wrench">
+    <xacro:u_bracket prefix="${prefix}" parent="${prefix}j2n6s300_wrench">
         <origin xyz="0.075 0 0.01525" rpy="${PI} 0 0"/>
     </xacro:u_bracket>
-    <xacro:kinect_wrist_connection num="1" parent_link="j2n6s300_wrench">
+    <xacro:kinect_wrist_connection prefix="${prefix}" num="1" parent_link="${prefix}j2n6s300_wrench">
         <origin xyz="0.025 -0.025 -0.005" rpy="${PI/2} 0 -${PI/2}"/>
     </xacro:kinect_wrist_connection>
-    <xacro:kinect_wrist_connection num="2" parent_link="j2n6s300_wrench">
+    <xacro:kinect_wrist_connection prefix="${prefix}" num="2" parent_link="${prefix}j2n6s300_wrench">
         <origin xyz="0.025 0.025 -0.005" rpy="${PI/2} ${PI} -${PI/2}"/>
     </xacro:kinect_wrist_connection>
     <!-- Azure Kinect -->
     <xacro:include filename="$(find oarbot_description)/urdf/microsoft/azure_kinect.urdf.xacro"/>
-    <xacro:azure_kinect parent_link="right_mount">
+    <xacro:azure_kinect prefix="${prefix}" parent_link="${prefix}right_mount">
         <origin xyz="0.006 0 -0.05" rpy="0 ${PI/2} 0" />
     </xacro:azure_kinect>
@@ -55,14 +56,14 @@
     <xacro:include filename="$(find oarbot_description)/urdf/hokuyo/hokuyo_ust.urdf.xacro"/>
     <!-- Front Sensor -->
-    <xacro:hokuyo_ust name="hokuyo_ust_front" parent_link="front_2_mount">
+    <xacro:hokuyo_ust prefix="${prefix}" name="hokuyo_ust_front" parent_link="${prefix}front_2_mount">
         <origin xyz="0.045 0 0" rpy="0 0 0"/>
     </xacro:hokuyo_ust>
     <!-- Rear Sensor -->
-    <xacro:hokuyo_ust name="hokuyo_ust_rear" parent_link="rear_2_mount">
+    <xacro:hokuyo_ust prefix="${prefix}" name="hokuyo_ust_rear" parent_link="${prefix}rear_2_mount">
         <origin xyz="-0.045 0 0" rpy="0 0 ${PI}"/>
     </xacro:hokuyo_ust>
     <!-- Microstrain IMU -->
     <xacro:include filename="$(find oarbot_description)/urdf/microstrain/microstrain_imu.urdf.xacro"/>
-    <xacro:microstrain_imu name="microstrain_imu" parent_link="default_mount">
+    <xacro:microstrain_imu prefix="${prefix}" name="microstrain_imu" parent_link="${prefix}default_mount">
         <origin xyz="0 0 0" rpy="0 0 0"/>
     </xacro:microstrain_imu>
