Commit message: Working oarbot_silver moveit2 with simulated data

File: src/oarbot_silver_moveit/config/oarbot_silver.ros2_control.xacro (robot description, xacro)
@@ -50,4 +50,46 @@
                 <state_interface name="velocity"/>
             </joint>
+            <joint name="j2n6s300_joint_finger_1">
+                <command_interface name="position"/>
+                <state_interface name="position">
+                  <param name="initial_value">${initial_positions['j2n6s300_joint_finger_1']}</param>
+                </state_interface>
+                <state_interface name="velocity"/>
+            </joint>
+            <joint name="j2n6s300_joint_finger_tip_1">
+                <command_interface name="position"/>
+                <state_interface name="position">
+                  <param name="initial_value">${initial_positions['j2n6s300_joint_finger_tip_1']}</param>
+                </state_interface>
+                <state_interface name="velocity"/>
+            </joint>
+            <joint name="j2n6s300_joint_finger_2">
+                <command_interface name="position"/>
+                <state_interface name="position">
+                  <param name="initial_value">${initial_positions['j2n6s300_joint_finger_2']}</param>
+                </state_interface>
+                <state_interface name="velocity"/>
+            </joint>
+            <joint name="j2n6s300_joint_finger_tip_2">
+                <command_interface name="position"/>
+                <state_interface name="position">
+                  <param name="initial_value">${initial_positions['j2n6s300_joint_finger_tip_2']}</param>
+                </state_interface>
+                <state_interface name="velocity"/>
+            </joint>
+            <joint name="j2n6s300_joint_finger_3">
+                <command_interface name="position"/>
+                <state_interface name="position">
+                  <param name="initial_value">${initial_positions['j2n6s300_joint_finger_3']}</param>
+                </state_interface>
+                <state_interface name="velocity"/>
+            </joint>
+            <joint name="j2n6s300_joint_finger_tip_3">
+                <command_interface name="position"/>
+                <state_interface name="position">
+                  <param name="initial_value">${initial_positions['j2n6s300_joint_finger_tip_3']}</param>
+                </state_interface>
+                <state_interface name="velocity"/>
+            </joint>
         </ros2_control>
     </xacro:macro>

Commit message: Update to use prefixed robot description

File: src/oarbot_silver_moveit/config/oarbot_silver.ros2_control.xacro (robot description, xacro)
@@ -8,85 +8,85 @@
                 <plugin>mock_components/GenericSystem</plugin>
             </hardware>
-            <joint name="j2n6s300_joint_1">
+            <joint name="oarbot_silver/j2n6s300_joint_1">
                 <command_interface name="position"/>
                 <state_interface name="position">
-                  <param name="initial_value">${initial_positions['j2n6s300_joint_1']}</param>
+                  <param name="initial_value">${initial_positions['oarbot_silver/j2n6s300_joint_1']}</param>
                 </state_interface>
                 <state_interface name="velocity"/>
             </joint>
-            <joint name="j2n6s300_joint_2">
+            <joint name="oarbot_silver/j2n6s300_joint_2">
                 <command_interface name="position"/>
                 <state_interface name="position">
-                  <param name="initial_value">${initial_positions['j2n6s300_joint_2']}</param>
+                  <param name="initial_value">${initial_positions['oarbot_silver/j2n6s300_joint_2']}</param>
                 </state_interface>
                 <state_interface name="velocity"/>
             </joint>
-            <joint name="j2n6s300_joint_3">
+            <joint name="oarbot_silver/j2n6s300_joint_3">
                 <command_interface name="position"/>
                 <state_interface name="position">
-                  <param name="initial_value">${initial_positions['j2n6s300_joint_3']}</param>
+                  <param name="initial_value">${initial_positions['oarbot_silver/j2n6s300_joint_3']}</param>
                 </state_interface>
                 <state_interface name="velocity"/>
             </joint>
-            <joint name="j2n6s300_joint_4">
+            <joint name="oarbot_silver/j2n6s300_joint_4">
                 <command_interface name="position"/>
                 <state_interface name="position">
-                  <param name="initial_value">${initial_positions['j2n6s300_joint_4']}</param>
+                  <param name="initial_value">${initial_positions['oarbot_silver/j2n6s300_joint_4']}</param>
                 </state_interface>
                 <state_interface name="velocity"/>
             </joint>
-            <joint name="j2n6s300_joint_5">
+            <joint name="oarbot_silver/j2n6s300_joint_5">
                 <command_interface name="position"/>
                 <state_interface name="position">
-                  <param name="initial_value">${initial_positions['j2n6s300_joint_5']}</param>
+                  <param name="initial_value">${initial_positions['oarbot_silver/j2n6s300_joint_5']}</param>
                 </state_interface>
                 <state_interface name="velocity"/>
             </joint>
-            <joint name="j2n6s300_joint_6">
+            <joint name="oarbot_silver/j2n6s300_joint_6">
                 <command_interface name="position"/>
                 <state_interface name="position">
-                  <param name="initial_value">${initial_positions['j2n6s300_joint_6']}</param>
+                  <param name="initial_value">${initial_positions['oarbot_silver/j2n6s300_joint_6']}</param>
                 </state_interface>
                 <state_interface name="velocity"/>
             </joint>
-            <joint name="j2n6s300_joint_finger_1">
+            <joint name="oarbot_silver/j2n6s300_joint_finger_1">
                 <command_interface name="position"/>
                 <state_interface name="position">
-                  <param name="initial_value">${initial_positions['j2n6s300_joint_finger_1']}</param>
+                  <param name="initial_value">${initial_positions['oarbot_silver/j2n6s300_joint_finger_1']}</param>
                 </state_interface>
                 <state_interface name="velocity"/>
             </joint>
-            <joint name="j2n6s300_joint_finger_tip_1">
+            <joint name="oarbot_silver/j2n6s300_joint_finger_tip_1">
                 <command_interface name="position"/>
                 <state_interface name="position">
-                  <param name="initial_value">${initial_positions['j2n6s300_joint_finger_tip_1']}</param>
+                  <param name="initial_value">${initial_positions['oarbot_silver/j2n6s300_joint_finger_tip_1']}</param>
                 </state_interface>
                 <state_interface name="velocity"/>
             </joint>
-            <joint name="j2n6s300_joint_finger_2">
+            <joint name="oarbot_silver/j2n6s300_joint_finger_2">
                 <command_interface name="position"/>
                 <state_interface name="position">
-                  <param name="initial_value">${initial_positions['j2n6s300_joint_finger_2']}</param>
+                  <param name="initial_value">${initial_positions['oarbot_silver/j2n6s300_joint_finger_2']}</param>
                 </state_interface>
                 <state_interface name="velocity"/>
             </joint>
-            <joint name="j2n6s300_joint_finger_tip_2">
+            <joint name="oarbot_silver/j2n6s300_joint_finger_tip_2">
                 <command_interface name="position"/>
                 <state_interface name="position">
-                  <param name="initial_value">${initial_positions['j2n6s300_joint_finger_tip_2']}</param>
+                  <param name="initial_value">${initial_positions['oarbot_silver/j2n6s300_joint_finger_tip_2']}</param>
                 </state_interface>
                 <state_interface name="velocity"/>
             </joint>
-            <joint name="j2n6s300_joint_finger_3">
+            <joint name="oarbot_silver/j2n6s300_joint_finger_3">
                 <command_interface name="position"/>
                 <state_interface name="position">
-                  <param name="initial_value">${initial_positions['j2n6s300_joint_finger_3']}</param>
+                  <param name="initial_value">${initial_positions['oarbot_silver/j2n6s300_joint_finger_3']}</param>
                 </state_interface>
                 <state_interface name="velocity"/>
             </joint>
-            <joint name="j2n6s300_joint_finger_tip_3">
+            <joint name="oarbot_silver/j2n6s300_joint_finger_tip_3">
                 <command_interface name="position"/>
                 <state_interface name="position">
-                  <param name="initial_value">${initial_positions['j2n6s300_joint_finger_tip_3']}</param>
+                  <param name="initial_value">${initial_positions['oarbot_silver/j2n6s300_joint_finger_tip_3']}</param>
                 </state_interface>
                 <state_interface name="velocity"/>
